Commit message: Ajout de la phase d'indentification.

File: motoman_hc10_support/urdf/hc10_gazebo.urdf (robot description, URDF)
Before this commit: robot motoman_hc10, 9 links, 8 joints
Joints:
- joint joint_6_t-tool0: origin xyz=0 0 -0.130 rpy=3.14159265359 0 0 -> xyz=0.063 0.004 0.216 rpy=3.14159265359 0 0

File: motoman_hc10_support/urdf/hc10_macro.xacro (robot description, xacro)
@@ -144,5 +144,5 @@
     </joint>
     <joint name="${prefix}joint_6_t-tool0" type="fixed">
-      <origin xyz="0 0 -0.130" rpy="${pi} 0 0"/>
+      <origin xyz="0.063 0.004 -0.216" rpy="${pi} 0 0"/>
       <parent link="${prefix}link_6_t"/>
       <child link="${prefix}tool0"/>
