Commit message: Modification repère outil

File: motoman_hc10_support/urdf/hc10_macro.xacro (robot description, xacro)
@@ -144,5 +144,5 @@
     </joint>
     <joint name="${prefix}joint_6_t-tool0" type="fixed">
-      <origin xyz="0.063 0.004 -0.216" rpy="${pi} 0 0"/>
+      <origin xyz="0.062 0.0 -0.211" rpy="${pi} 0 0"/>
       <parent link="${prefix}link_6_t"/>
       <child link="${prefix}tool0"/>
